File: KICAD/SCREEN/SCREEN_V1.2/ESP-12E.kicad_sch (KiCad schematic)
At the start: 29 parts, among them J10 Conn_01x06_Socket, J13 Conn_01x04_Socket, J14 Conn_01x03_Pin, J18 Conn_01x02_Pin, J5 Conn_01x02_Pin, SW5 FLASH_BOOT | UART SWT, U4 ESP-12E

Commit message: .
Changed lines of the file:
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@@
 (kicad_sch
-	(version 20231120)
+	(version 20250114)
 	(generator "eeschema")
-	(generator_version "8.0")
+	(generator_version "9.0")
 	(paper "A4")
 	(junction
