File: KICAD/SCREEN/SCREEN_V1.2/SCREEN_VERSION_1.2.kicad_pcb (KiCad board)
At the start: 6 copper layers, 169 x 106.5 mm, 147 parts, among them J1 Conn_01x40, J10 Conn_01x06_Socket, J11 Conn_01x02_Socket, J12 Conn_01x02_Socket, J13 Conn_01x04_Socket, J14 Conn_01x03_Pin, J15 Conn_01x04_Socket, J16 Conn_01x02_Socket, J17 RJ45, J18 Conn_01x02_Pin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

Commit message: .
Parts:
- added D14: C106DGOS-ND, Package_SIP:SIP3_11.6x8.5mm, F.Cu at (231.4, 77.2)
- added F1: Polyfuse, Fuse:Fuse_1206_3216Metric, F.Cu at (215.5, 66.6)
- added R27: 4k, Resistor_SMD:R_0402_1005Metric, F.Cu at (216.8, 78.5)
- added R28: 10k, Resistor_SMD:R_0402_1005Metric, F.Cu at (214.0, 78.5)
- added R29: 1k, Resistor_SMD:R_0402_1005Metric, F.Cu at (217.5, 76.4)
- added R30: 100, Resistor_SMD:R_0402_1005Metric, F.Cu at (219.4, 76.4)
- added R31: 10k, Resistor_SMD:R_0402_1005Metric, F.Cu at (221.8, 75.1)
- added U10: TL431DBZ, Package_TO_SOT_SMD:SOT-23, F.Cu at (216.6, 82.8)
- moved G*** 81.0 mm to (112.8, 139.7)
- moved J2 17.5 mm to (211.5, 87.8)
- moved J13 16.7 mm to (222.9, 153.3)
- moved J17 11.9 mm to (228.6, 96.7)
- moved C53 9.00 mm to (216.8, 116.2)
- moved C54 9.00 mm to (215.5, 138.2)
- moved C57 9.00 mm to (222.8, 117.2)
- moved C58 9.00 mm to (227.0, 116.4)
- moved C59 9.00 mm to (217.7, 137.7)
- moved C60 9.00 mm to (214.6, 116.2)
- moved D1 9.00 mm to (227.6, 113.9)
- moved D3 9.00 mm to (222.2, 114.4)
- moved D4 9.00 mm to (220.2, 139.2)
- moved D5 9.00 mm to (222.5, 139.2)
- moved J10 9.00 mm to (219.1, 108.8)
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- renumbered SW1 to BOOT_SWT, SW4 to BYPASS_REG_SWT, SW2 to NRST_SWT, SW3 to PDR_SWT
Connections:
- U14 pad 1: +12V -> Net-(U14-VIN)
Routing:
- net +12V: track 499.9 -> 512.3 mm
- net Net-(J10-Pin_4): track 57.4 -> 69.5 mm, vias 1 -> 2
- net Net-(D14-G): track 0.00 -> 11.6 mm
- net /ESP-12E/UART_TX: track 17.3 -> 6.69 mm
- net /ESP-12E/ESP_RX: track 113.7 -> 123.4 mm, vias 3 -> 4
- net /ESP-12E/EN: track 73.5 -> 81.3 mm
- net GND: track 189.1 -> 197.0 mm, vias 112 -> 114
- net Net-(U10-K): track 0.00 -> 7.08 mm
- net /ESP-12E/RST: track 77.1 -> 83.7 mm
- net Net-(U14-VIN): track 0.00 -> 5.97 mm
- net Net-(U10-REF): track 0.00 -> 5.42 mm
- net Net-(D14-K): track 0.00 -> 5.30 mm
- net Net-(J2-Pin_2): track 10.9 -> 6.05 mm
- net /ESP-12E/RTS: track 73.7 -> 77.5 mm
- net /ESP-12E/CTS: track 48.3 -> 52.0 mm
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Other:
- board size 169 x 106.5 mm -> 168.7 x 106.5 mm
- board text added: "1"
- board text added: "CTS"
- board text added: "GND"
- board text added: "RTS"
- board text added: "RXD"
- board text added: "TXD"
- board text added: "VCC"
