File: KICAD/SCREEN/SCREEN_V1.2/STM32F469IIT6.kicad_sch (KiCad schematic)
At the start: 47 parts, among them J11 Conn_01x02_Socket, J12 Conn_01x02_Socket, J15 Conn_01x04_Socket, J16 Conn_01x02_Socket, J17 RJ45, J2 Conn_01x02_Socket, J3 Conn_01x05_Pin, SW1 BOOT0_SWT, SW2 NRST_SWT, SW3 PDR_ON SWT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

Commit message: .
Changed lines of the file:
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@@
 (kicad_sch
-	(version 20231120)
+	(version 20250114)
 	(generator "eeschema")
-	(generator_version "8.0")
+	(generator_version "9.0")
 	(paper "A3")
 	(junction
